File: H-bridge_double.sch (EAGLE design)
At the start: 34 parts, among them Q1 2N2222A, Q2 2N2222A, Q3 2N2907, Q4 2N2907, Q5 2N2222A, Q6 2N2222A, Q7 2N2907, Q8 2N2907, X1 22-23-2051, X3 22-23-2051

Commit message: Eagle CAD for Dual H-bridge
Parts:
- added 5-V, 5V: LSP10, solpad:LSP10
Connections:
- new net N$19: 5V.MP, ARDUINO_POWER-2.S, R5.A
- net N$15: now also 5-V.MP; no longer ARDUINO_POWER-2.S, R5.A
Changed lines of the file:
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@@
 <part name="R10" library="pot" deviceset="TRIM_EU-" device="CA6V"/>
 <part name="VCC" library="con-lstb" deviceset="MA03-1" device=""/>
+<part name="5V" library="solpad" deviceset="LSP10" device=""/>
+<part name="5-V" library="solpad" deviceset="LSP10" device=""/>
 </parts>
 <sheets>
@@
 <instance part="R10" gate="1" x="162.56" y="-2.54"/>
 <instance part="VCC" gate="G$1" x="66.04" y="106.68" rot="R270"/>
+<instance part="5V" gate="1" x="86.36" y="-22.86" rot="R270"/>
+<instance part="5-V" gate="1" x="172.72" y="-12.7" rot="R270"/>
 </instances>
 <busses>
@@
 <net name="N$15" class="0">
 <segment>
-<pinref part="R5" gate="1" pin="A"/>
-<wire x1="66.04" y1="-7.62" x2="66.04" y2="-15.24" width="0.1524" layer="91"/>
-<pinref part="ARDUINO_POWER" gate="-2" pin="S"/>
-<wire x1="66.04" y1="-15.24" x2="78.74" y2="-15.24" width="0.1524" layer="91"/>
-<wire x1="78.74" y1="-15.24" x2="83.82" y2="-15.24" width="0.1524" layer="91"/>
-<wire x1="78.74" y1="-15.24" x2="78.74" y2="-35.56" width="0.1524" layer="91"/>
-<wire x1="78.74" y1="-35.56" x2="162.56" y2="-35.56" width="0.1524" layer="91"/>
 <pinref part="R10" gate="1" pin="A"/>
-<wire x1="162.56" y1="-35.56" x2="162.56" y2="-7.62" width="0.1524" layer="91"/>
+<wire x1="162.56" y1="-12.7" x2="162.56" y2="-7.62" width="0.1524" layer="91"/>
+<wire x1="170.18" y1="-12.7" x2="162.56" y2="-12.7" width="0.1524" layer="91"/>
+<pinref part="5-V" gate="1" pin="MP"/>
 </segment>
 </net>
@@
 </segment>
 </net>
+<net name="N$19" class="0">
+<segment>
+<pinref part="ARDUINO_POWER" gate="-2" pin="S"/>
+<wire x1="83.82" y1="-22.86" x2="83.82" y2="-15.24" width="0.1524" layer="91"/>
+<junction x="83.82" y="-15.24"/>
+<pinref part="R5" gate="1" pin="A"/>
+<wire x1="66.04" y1="-7.62" x2="66.04" y2="-15.24" width="0.1524" layer="91"/>
+<wire x1="66.04" y1="-15.24" x2="83.82" y2="-15.24" width="0.1524" layer="91"/>
+<pinref part="5V" gate="1" pin="MP"/>
+</segment>
+</net>
